File: kicad/adaptateur_capteur/adaptateur_capteur.sch (KiCad schematic (older format))
At the start: 4 parts, among them J1 AudioJack4, U1 BME680

Commit message: Dump v0.2
As time was of the essence, and I was developing this alone, versioning was not done (shame!)
This version is more of a dump of all code / some unfinished schematics, and (not always translate) docs
It should works fine, but it definitely not bug-free as for now.
Parts:
- U1: symbol sechoir_solaire:BME680 -> adaptateur_capteur:BME680
Changed lines of the file:
@@
 EESchema Schematic File Version 4
-EELAYER 29 0
+EELAYER 30 0
 EELAYER END
 $Descr A4 11693 8268
@@
 $EndDescr
 $Comp
-L sechoir_solaire:BME680 U1
+L adaptateur_capteur:BME680 U1
 U 1 1 5F2C0F60
 P 1850 2650
